File: Boards/GSat/GSat board/GSat board.kicad_pcb (KiCad board)
At the start: 2 copper layers, 100 x 140 mm, 59 parts, among them IC1 LTC4418IUF#PBF, IC2 MCP23017-E_SP, J1 B3B-XH-A_LF__SN_, J10 Conn_01x05_Pin, J11 Conn_01x06_Pin, J12 XT30UPB-F, J13 B4B-XH-A_LF__SN_, J14 B4B-XH-A_LF__SN_, J15 B4B-XH-A_LF__SN_, J16 B4B-XH-A_LF__SN_, J2 XT30UPB-F, J3 B3B-XH-A_LF__SN_, J4 B3B-XH-A_LF__SN_, Q1 PMOS, Q2 PMOS, Q3 PMOS, Q4 PMOS, U1 TMC2209_SILENTSTEPSTICK, U10 ST1L05APU33R, U2 TMC2209_SILENTSTEPSTICK, U3 E28-2G4M27SX, U4 E28-2G4M27SX, U5 MAX485_MODULE_5V_LOGIC_TLL_TO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

Commit message: Revert "GSPOT"
This reverts commit 8c379314ca4fbea904d10af8cef34905ce442d4e.
Parts:
- removed J1, J3, J4: B3B-XH-A_LF__SN_, B3B-XH-A_LF__SN:B3BXHALFSN
- added TP5: TestPoint, TestPoint:TestPoint_Pad_2.0x2.0mm, F.Cu at (244.5, 69.5)
- moved R14 145.5 mm to (132.9, 48.6), turned to 0 degrees
- moved R2 93.8 mm to (139.3, 45.0), turned to 0 degrees
- moved R3 89.8 mm to (139.3, 47.5), turned to 0 degrees
- moved R11 87.0 mm to (132.9, 42.1), turned to 0 degrees
- moved R13 57.9 mm to (132.9, 46.4), turned to 0 degrees
- moved R12 44.1 mm to (132.9, 44.3), turned to 0 degrees
- moved C39 2.70 mm to (231.2, 41.1), turned to 0 degrees
- moved U10 2.58 mm to (232.0, 38.0)
- moved U6 2.58 mm to (243.3, 54.3)
- moved C37 2.58 mm to (234.8, 38.9)
- moved C40 2.58 mm to (236.3, 38.8)
- moved TP2 2.58 mm to (231.5, 43.3)
- moved R1 2.03 mm to (220.8, 149.5)
- moved U5 2.03 mm to (220.8, 125.3)
- moved J13 1.50 mm to (170.2, 82.2)
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Connections:
- A1 pad 33: GND -> unconnected-(A1-AGND-Pad33)
- C39 pad 2: +3.3V IC -> +3.3V
- TP2 pad 1: +3.3V IC -> +3.3V
- U1 pad 16: +3.3V IC -> +3.3V
- U1 pad 2: +3.3V IC -> +3.3V
- U10 pad 2: +3.3V IC -> +3.3V
- U2 pad 16: +3.3V IC -> +3.3V
- U2 pad 2: +3.3V IC -> +3.3V
Routing:
- net /CS_MSD: track 43.5 -> 51.3 mm
- net +24V: track 30.6 -> 37.2 mm
- net /RS_TX: track 31.7 -> 29.7 mm
- net /RS_RX: track 25.6 -> 23.6 mm
- net Net-(U1-M1B): track 10.3 -> 12.2 mm
- net Net-(U2-M1B): track 10.3 -> 12.1 mm
- net Net-(U1-M2B): track 8.55 -> 10.0 mm
- net Net-(U1-M2A): track 7.77 -> 9.27 mm
- net Net-(U1-M1A): track 7.75 -> 9.25 mm
- net Net-(U2-M2A): track 7.75 -> 9.17 mm
- net Net-(U2-M2B): track 8.53 -> 9.95 mm
- net Net-(U2-M1A): track 7.73 -> 9.15 mm
- net /RS_ENABLE: track 34.0 -> 34.5 mm
