File: Boards/GSat/GSat board/GSat board.kicad_pcb (KiCad board)
At the start: 2 copper layers, 100 x 140 mm, 63 parts, among them IC1 LTC4418IUF#PBF, IC2 MCP23017-E_SP, IC3 SP3485CN-L_TR, J1 B3B-XH-A_LF__SN_, J10 Conn_01x05_Pin, J11 Conn_01x06_Pin, J12 XT30UPB-F, J13 B4B-XH-A_LF__SN_, J14 B4B-XH-A_LF__SN_, J15 B4B-XH-A_LF__SN_, J16 B4B-XH-A_LF__SN_, J2 XT30UPB-F, J3 B3B-XH-A_LF__SN_, J4 B3B-XH-A_LF__SN_, Q1 PMOS, Q2 PMOS, Q3 PMOS, Q4 PMOS, U1 TMC2209_SILENTSTEPSTICK, U10 ST1L05APU33R, U2 TMC2209_SILENTSTEPSTICK, U3 E28-2G4M27SX, U4 E28-2G4M27SX, U5 MAX485_MODULE_5V_LOGIC_TLL_TO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

Commit message: GSAT REORGANIZED AND TRACED (mostly)
insert here the entire shrek script
Parts:
- removed C37, C39: 4.7uF, Capacitor-0402:Capacitor_0402
- removed C40: 1uF, Capacitor-0402:Capacitor_0402
- removed C41: 1nF, Capacitor-0402:Capacitor_0402
- removed C42, C43, C44, C45, C46: 100nF, Capacitor-0402:Capacitor_0402
- removed C47: 220uF, Capacitor-0402:Capacitor_0402
- removed D1, D2: SMBJ24CA, SMBJ24CA:DIOM5436X244N
- removed F1, F2: 0ABB-6000-TM, 0ABB-6000-TM:0ABB6000TM
- removed IC1: LTC4418IUF#PBF, LTC4418:QFN50P400X400X80-21N-D
- removed J12, J2: XT30UPB-F, XT30UPB-F:XT30UPBF
- removed Q1, Q2, Q3, Q4: PMOS, Package_TO_SOT_SMD:TO-252-3_TabPin2
- removed R1: 1K, Resistor_SMD:R_0603_1608Metric_Pad0.98x0.95mm_HandSolder
- removed R10, R5: 9.31K, Resistor_SMD:R_0603_1608Metric_Pad0.98x0.95mm_HandSolder
- removed R15, R7: 39.6K, Resistor_SMD:R_0603_1608Metric_Pad0.98x0.95mm_HandSolder
- removed R3: 10K, Resistor_SMD:R_0603_1608Metric_Pad0.98x0.95mm_HandSolder
- removed R4, R9: 1M, Resistor_SMD:R_0603_1608Metric_Pad0.98x0.95mm_HandSolder
- removed TP2, TP3, TP4: TestPoint, TestPoint:TestPoint_Pad_2.0x2.0mm
- removed U10: ST1L05APU33R, LDO ST1L05A:DFN_5APU33R_STM
- removed U5: MAX485_MODULE_5V_LOGIC_TLL_TO_RS-485_CONVERTER, MAX485Module:MODULE_MAX485_MODULE_5V_LOGIC_TLL_TO_RS-485_CONVERTER
- added J5: 1723163304, 1723163304:MOLEX_1723163304, F.Cu at (193.0, 97.5)
- added REF**: MountingHole_3.2mm_M3_DIN965, MountingHole:MountingHole_3.2mm_M3_DIN965, F.Cu at (176.0, 73.0)
- added REF**: MountingHole_3.2mm_M3_DIN965, MountingHole:MountingHole_3.2mm_M3_DIN965, F.Cu at (176.0, 152.0)
- added REF**: MountingHole_3.2mm_M3_DIN965, MountingHole:MountingHole_3.2mm_M3_DIN965, F.Cu at (241.0, 94.0)
- C4, C5: footprint Capacitor-0402:Capacitor_0402 -> Capacitor_SMD:C_0603_1608Metric_Pad1.08x0.95mm_HandSolder
- R11, R12, R13, R14, R6, R8: footprint Resistor-0402:RES_0402 -> Resistor_SMD:R_0603_1608Metric_Pad0.98x0.95mm_HandSolder
- U4: value E28-2G4M27SX -> LD1117S33TR_SOT223; footprint Radio_Module_PST:Radio_Module_PST -> Package_TO_SOT_SMD:SOT-223-3_TabPin2
- moved IC3 94.1 mm to (222.4, 119.2), turned to 90 degrees
- moved R16 90.4 mm to (218.8, 114.4)
- moved R17 86.3 mm to (222.3, 114.4)
- moved R18 82.1 mm to (225.8, 114.4)
- moved U4 55.0 mm to (233.0, 99.0), turned to -90 degrees
- moved J3 53.2 mm to (214.2, 76.5), turned to 90 degrees
- moved U6 47.3 mm to (215.0, 94.1), turned to 0 degrees
- moved R12 44.3 mm to (208.7, 75.0), turned to -90 degrees
- moved J4 35.4 mm to (215.0, 64.0), turned to 90 degrees
- moved R13 26.7 mm to (209.5, 63.0), turned to -90 degrees
- moved U3 19.9 mm to (232.4, 69.5)
- moved R2 18.8 mm to (244.0, 85.0), turned to 180 degrees
- moved IC2 13.5 mm to (222.5, 141.5)
- moved R14 13.3 mm to (229.5, 150.5)
- moved J11 13.0 mm to (240.5, 103.0)
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Connections:
- A1 pad 22: /CS_OMNI -> /EXP INTERRUPT
- A1 pad 27: /OMNI_BUSY -> unconnected-(A1-GPIO21-Pad27)
- A1 pad 29: /OMNI_DIO1 -> unconnected-(A1-GPIO22-Pad29)
- A1 pad 36: +3.3V -> unconnected-(A1-3V3-Pad36)_1
- IC2 pad 26: /OMNI_NRESET -> unconnected-(IC2-GPA5-Pad26)
- IC2 pad 27: /OMNI_RX_EN -> unconnected-(IC2-GPA6-Pad27)
- IC2 pad 28: /OMNI_TX_EN -> unconnected-(IC2-GPA7-Pad28)
- U1 pad 16: +3.3V IC -> +3.3V
- U1 pad 2: +3.3V IC -> +3.3V
- U2 pad 16: +3.3V IC -> +3.3V
- U4 pad 1: +3.3V -> GND
- U4 pad 2: GND -> +3.3V
- U4 pad 3: /RADIO MISO -> +5V
Routing:
- net /LimitSwitch3: track 0.00 -> 90.0 mm, vias 0 -> 2
- net /RADIO MISO: track 0.00 -> 85.3 mm, vias 0 -> 2
- net /RADIO CLK: track 0.00 -> 83.4 mm, vias 0 -> 4
- net /LimitSwitch2: track 0.00 -> 80.4 mm, vias 0 -> 2
- net /RADIO MOSI: track 0.00 -> 79.3 mm, vias 0 -> 2
- net /UNI_TX_EN: track 0.00 -> 76.8 mm, vias 0 -> 2
- net /CS_UNI: track 0.00 -> 71.9 mm, vias 0 -> 1
- net /UNI_NRESET: track 0.00 -> 71.3 mm, vias 0 -> 1
- net /Driver2 VREF: track 1.61 -> 71.1 mm, vias 0 -> 1
- net /Driver1 Dir: track 22.2 -> 88.9 mm, vias 1 -> 2
- net /LimitSwitch1: track 0.00 -> 63.4 mm
- net /Driver2 MS1: track 29.8 -> 91.3 mm, vias 1 -> 2
- net /Driver1 MS2: track 10.4 -> 70.3 mm, vias 1 -> 2
- net /RS_B: track 0.00 -> 59.2 mm, vias 0 -> 3
- net /Driver2 MS2: track 32.0 -> 90.5 mm, vias 1 -> 2
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Other:
- board size 100 x 140 mm -> 75 x 108 mm

Commit message: GSPOT update
Parts:
- removed C4, C5: 100n, Capacitor_SMD:C_0603_1608Metric_Pad1.08x0.95mm_HandSolder
- removed J11: Conn_01x06_Pin, Connector_PinSocket_2.54mm:PinSocket_1x06_P2.54mm_Vertical
- removed R6, R8: 1k, Resistor_SMD:R_0603_1608Metric_Pad0.98x0.95mm_HandSolder
- added C1: 100n, Capacitor_SMD:C_0603_1608Metric_Pad1.08x0.95mm_HandSolder, F.Cu at (201.5, 92.5)
- added C2: 100n, Capacitor_SMD:C_0603_1608Metric_Pad1.08x0.95mm_HandSolder, F.Cu at (180.0, 89.5)
- added C3: 100n, Capacitor_SMD:C_0603_1608Metric_Pad1.08x0.95mm_HandSolder, F.Cu at (196.4, 56.5)
- added C44: 470u, Capacitor_SMD:CP_Elec_10x10, F.Cu at (195.0, 100.0)
- added C7: 100u, Capacitor_SMD:CP_Elec_6.3x7.7, F.Cu at (176.3, 94.5)
- added C9: 100u, Capacitor_SMD:CP_Elec_6.3x7.7, F.Cu at (204.8, 59.5)
- added D1: D_Zener, Diode_SMD:D_SMB, F.Cu at (219.8, 107.5)
- added F1: 0ABB-6000-TM, 0ABB-6000-TM:0ABB6000TM, F.Cu at (187.4, 96.5)
- added R7: 10k, Resistor_SMD:R_0603_1608Metric_Pad0.98x0.95mm_HandSolder, F.Cu at (198.0, 92.6)
- added R9: 10k, Resistor_SMD:R_0603_1608Metric_Pad0.98x0.95mm_HandSolder, F.Cu at (180.0, 75.4)
- moved J4 11.7 mm to (204.0, 68.0), turned to 0 degrees
- moved J3 10.8 mm to (204.0, 80.0), turned to 0 degrees
- moved J5 10.5 mm to (184.0, 103.0)
- moved R13 10.5 mm to (205.0, 72.5), turned to 180 degrees
- moved U2 8.86 mm to (189.5, 65.5)
- moved J10 8.55 mm to (232.0, 140.9)
- moved REF** 6.18 mm to (235.0, 92.5)
- moved R2 6.00 mm to (238.0, 85.0)
- moved U3 5.90 mm to (226.5, 69.5)
- moved R12 3.74 mm to (205.0, 74.5), turned to 180 degrees
- moved R14 3.64 mm to (226.0, 149.5), turned to -90 degrees
- moved IC3 3.37 mm to (219.0, 119.1)
- moved R16 3.25 mm to (215.5, 114.3)
- moved R17 3.25 mm to (219.0, 114.3)
- moved R18 3.25 mm to (222.5, 114.3)
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Connections:
- A1 pad 16: /MSD MISO -> /TMC EN
- A1 pad 17: /CS_MSD -> unconnected-(A1-GPIO13-Pad17)
- A1 pad 19: /MSD CLK -> unconnected-(A1-GPIO14-Pad19)
- A1 pad 20: /MSD MOSI -> unconnected-(A1-GPIO15-Pad20)
- A1 pad 31: /Driver1 VREF -> unconnected-(A1-GPIO26_ADC0-Pad31)
- A1 pad 32: /Driver2 VREF -> unconnected-(A1-GPIO27_ADC1-Pad32)
- A1 pad 34: /GPS PPS -> unconnected-(A1-GPIO28_ADC2-Pad34)
- A1 pad 35: GND -> unconnected-(A1-ADC_VREF-Pad35)
- J5 pad 1: +24V -> Net-(F1-Pad2)
- U1 pad 16: +3.3V -> /TMC EN
- U1 pad 18: Net-(U1-DIAG) -> unconnected-(U1-DIAG-Pad18)
- U1 pad 8: +24V -> +12V
- U2 pad 16: +3.3V -> /TMC EN
- U2 pad 18: Net-(U2-DIAG) -> unconnected-(U2-DIAG-Pad18)
- U2 pad 2: +3.3V IC -> +3.3V
- U2 pad 8: +24V -> +12V
- U6 pad 1: +24V -> +12V
Routing:
- net /EXP INTERRUPT: track 0.00 -> 71.5 mm, vias 0 -> 2
- net /Driver2 VREF: track 71.1 -> 0.00 mm, vias 1 -> 0
- net /GPS PPS: track 68.6 -> 0.00 mm, vias 2 -> 0
- net /RADIO MISO: track 85.3 -> 31.9 mm, vias 2 -> 1
- net /Driver1 VREF: track 50.8 -> 0.00 mm, vias 1 -> 0
- net /LimitSwitch3: track 90.0 -> 42.3 mm
- net /RADIO MOSI: track 79.3 -> 32.1 mm, vias 2 -> 1
- net /Driver2 MS1: track 91.3 -> 52.2 mm
- net /Driver2 Dir: track 88.4 -> 50.1 mm
- net /CS_MSD: track 38.2 -> 0.00 mm, vias 2 -> 0
- net /LimitSwitch2: track 80.4 -> 44.6 mm
- net /MSD MISO: track 33.7 -> 0.00 mm
- net /Driver1 Dir: track 88.9 -> 57.6 mm
- net /MSD MOSI: track 30.9 -> 0.00 mm
- net /MSD CLK: track 30.7 -> 0.00 mm
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Other:
- board size 75 x 108 mm -> 69 x 106 mm

Commit message: GSPOT PCB (almost final)
apenas finalizar uma feature e detalhes
Parts:
- removed IC2: MCP23017-E_SP, MCP23017:DIP794W56P254L3486H508Q28N
- removed R14: 10k, Resistor_SMD:R_0603_1608Metric_Pad0.98x0.95mm_HandSolder
- added C5: 100n, Capacitor_SMD:C_0603_1608Metric_Pad1.08x0.95mm_HandSolder, F.Cu at (247.7, 73.8)
- added J17: B4B-XH-A_LF__SN_, B4B-XH-A_LF__SN_:B4BXHALFSN, F.Cu at (202.0, 140.6)
- added J2: 172298-1104, 1723163304:172298-YY04, F.Cu at (180.5, 105.5)
- added J6: B2B-XH-A-M_LF__SN_, B2B-XH-A-M_LF__SN_:B2BXHAMLFSN, F.Cu at (175.0, 133.5)
- added J7: B2B-XH-A-M_LF__SN_, B2B-XH-A-M_LF__SN_:B2BXHAMLFSN, F.Cu at (186.2, 140.5)
- added J8: B2B-XH-A-M_LF__SN_, B2B-XH-A-M_LF__SN_:B2BXHAMLFSN, F.Cu at (176.7, 140.5)
- added R20: 1k, Resistor_SMD:R_0603_1608Metric_Pad0.98x0.95mm_HandSolder, F.Cu at (198.4, 112.0)
- added R21: 10k, Resistor_SMD:R_0603_1608Metric_Pad0.98x0.95mm_HandSolder, F.Cu at (247.7, 83.8)
- D1: value D_Zener -> SMAJ14A
- F1: value 0ABB-6000-TM -> 0680L4000-05; footprint 0ABB-6000-TM:0ABB6000TM -> Fuse:Fuse_2512_6332Metric
- J5: value 1723163304 -> B2B-XH-A-M_LF__SN_; footprint 1723163304:MOLEX_1723163304 -> B2B-XH-A-M_LF__SN_:B2BXHAMLFSN
- R11: value 10k -> 6.8k
- R12: value 10k -> 1k
- R13: value 10k -> 22k
- moved R11 75.5 mm to (247.7, 76.3), turned to 0 degrees
- moved J15 53.0 mm to (235.2, 140.5), turned to 180 degrees
- moved R13 43.6 mm to (247.7, 81.3), turned to 0 degrees
- moved R12 42.9 mm to (247.7, 78.8), turned to 0 degrees
- moved J16 38.4 mm to (218.6, 140.5), turned to 180 degrees
- moved J10 31.6 mm to (227.9, 109.5), turned to 90 degrees
- moved J5 30.5 mm to (183.0, 133.5), turned to 90 degrees
- moved REF** 28.0 mm to (175.5, 124.0)
- moved R18 19.8 mm to (204.5, 106.0)
- moved R17 16.6 mm to (203.2, 109.5), turned to 90 degrees
- moved A1 15.4 mm to (213.5, 124.5), turned to -90 degrees
- moved IC3 14.6 mm to (208.0, 109.5), turned to 180 degrees
- moved R16 13.7 mm to (202.0, 112.0)
- moved C1 9.86 mm to (201.5, 102.4), turned to -90 degrees
- moved J1 5.97 mm to (175.0, 117.5), turned to 0 degrees
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Connections:
- A1 pad 10: /I2C#2 SCL -> /UNI_TX_EN
- A1 pad 14: /UNI_BUSY -> /RS_ENABLE
- A1 pad 15: /UNI_DIO1 -> /Driver2 Step
- A1 pad 16: /TMC EN -> /TMC TX UART
- A1 pad 17: unconnected-(A1-GPIO13-Pad17) -> /TMC RX UART
- A1 pad 19: unconnected-(A1-GPIO14-Pad19) -> /TMC EN
- A1 pad 20: unconnected-(A1-GPIO15-Pad20) -> /Driver1 Step
- A1 pad 21: /RADIO MISO -> /I2C#1 SDA
- A1 pad 22: /EXP INTERRUPT -> /I2C#1 SCL
- A1 pad 24: /RADIO CLK -> /Driver2 Dir
- A1 pad 25: /RADIO MOSI -> /Driver1 Dir
- A1 pad 26: /CS_UNI -> /UNI_DIO1
- A1 pad 27: unconnected-(A1-GPIO21-Pad27) -> /UNI_NRESET
- A1 pad 29: unconnected-(A1-GPIO22-Pad29) -> /UNI_BUSY
- A1 pad 31: unconnected-(A1-GPIO26_ADC0-Pad31) -> /I2C#2 SDA
- A1 pad 32: unconnected-(A1-GPIO27_ADC1-Pad32) -> /I2C#2 SCL
- A1 pad 34: unconnected-(A1-GPIO28_ADC2-Pad34) -> /LimitSense
- A1 pad 4: /Driver1 Step -> /RADIO CLK
- A1 pad 5: /Driver2 Step -> /RADIO MOSI
- A1 pad 6: /I2C#1 SDA -> /RADIO MISO
- A1 pad 7: /I2C#1 SCL -> /CS_UNI
- A1 pad 9: /I2C#2 SDA -> /UNI_RX_EN
- J1 pad 1: +3.3V -> /LimitSense
- J1 pad 2: /LimitSwitch1 -> unconnected-(J1-Pad2)
- J1 pad 3: GND -> Net-(J1-Pad3)
- J15 pad 2: /I2C#1 SDA -> /I2C#2 SDA
- J15 pad 3: /I2C#1 SCL -> /I2C#2 SCL
- J3 pad 1: +3.3V -> /LimitSense
- J3 pad 2: /LimitSwitch2 -> unconnected-(J3-Pad2)
- J3 pad 3: GND -> Net-(J3-Pad3)
- J4 pad 1: +3.3V -> /LimitSense
- J4 pad 2: /LimitSwitch3 -> unconnected-(J4-Pad2)
- J4 pad 3: GND -> Net-(J4-Pad3)
- J5 pad 1: Net-(F1-Pad2) -> +5V
- J5 pad 2: GND -> Net-(J5-Pad2)
- R11 pad 1: /LimitSwitch1 -> GND
- R11 pad 2: +3.3V -> Net-(J3-Pad3)
- R12 pad 1: /LimitSwitch2 -> GND
- R12 pad 2: +3.3V -> Net-(J1-Pad3)
- R13 pad 1: /LimitSwitch3 -> GND
- R13 pad 2: +3.3V -> Net-(J4-Pad3)
- U1 pad 12: unconnected-(U1-UART-Pad12) -> /TMC RX UART
- U1 pad 14: /Driver1 MS2 -> GND
- U1 pad 15: /Driver1 MS1 -> GND
- U2 pad 12: unconnected-(U2-UART-Pad12) -> /TMC RX UART
- U2 pad 14: /Driver2 MS2 -> GND
- U2 pad 15: /Driver2 MS1 -> +3.3V
Routing:
- net +3.3V: track 4.65 -> 254.0 mm, vias 0 -> 4
- net +12V: track 0.00 -> 123.7 mm
- net +5V: track 0.00 -> 122.8 mm
- net /Driver2 MS2: track 86.9 -> 0.00 mm, vias 2 -> 0
- net /EXP INTERRUPT: track 71.5 -> 0.00 mm, vias 2 -> 0
- net /Driver1 MS2: track 60.9 -> 0.00 mm, vias 2 -> 0
- net /LimitSwitch1: track 59.8 -> 0.00 mm
- net /Driver1 MS1: track 56.8 -> 0.00 mm, vias 2 -> 0
- net /TMC EN: track 0.21 -> 57.0 mm
- net /Driver2 MS1: track 52.2 -> 0.00 mm, vias 2 -> 0
- net /TMC RX UART: track 0.00 -> 49.4 mm
- net /LimitSwitch2: track 44.6 -> 0.00 mm, vias 2 -> 0
- net /LimitSwitch3: track 42.3 -> 0.00 mm, vias 2 -> 0
- net /Driver2 Step: track 87.7 -> 46.3 mm, vias 3 -> 0
- net /I2C#1 SCL: track 48.0 -> 9.27 mm, vias 1 -> 0
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- added copper zone on B.Cu, net GND
- added copper zone on F.Cu, net GND
Other:
- board size 69 x 106 mm -> 70 x 90 mm

Commit message: RSPOT board (FINAL) (?)
Parts:
- removed J1, J3, J4: B3B-XH-A_LF__SN_, B3B-XH-A_LF__SN:B3BXHALFSN
- added J11: B2B-XH-A-M_LF__SN_, B2B-XH-A-M_LF__SN_:B2BXHAMLFSN, F.Cu at (205.5, 76.0)
- added J12: B2B-XH-A-M_LF__SN_, B2B-XH-A-M_LF__SN_:B2BXHAMLFSN, F.Cu at (175.5, 117.0)
- added J9: B2B-XH-A-M_LF__SN_, B2B-XH-A-M_LF__SN_:B2BXHAMLFSN, F.Cu at (205.5, 68.0)
- C1, C2, C3, C5: footprint Capacitor_SMD:C_0603_1608Metric_Pad1.08x0.95mm_HandSolder -> Capacitor_SMD:C_0805_2012Metric_Pad1.18x1.45mm_HandSolder
- R11, R12, R13, R18, R2, R20, R21, R7, R9: footprint Resistor_SMD:R_0603_1608Metric_Pad0.98x0.95mm_HandSolder -> Resistor_SMD:R_0805_2012Metric_Pad1.20x1.40mm_HandSolder
- moved R13 72.1 mm to (184.0, 115.0), turned to 180 degrees
- moved R11 39.1 mm to (209.0, 82.0), turned to 90 degrees
- moved R12 36.8 mm to (211.0, 82.0), turned to 90 degrees
- moved C5 21.2 mm to (232.0, 88.0), turned to 90 degrees
- moved R21 19.7 mm to (233.0, 97.0)
- moved R20 0.41 mm to (198.0, 112.0)
- moved R18 0.30 mm to (204.5, 105.7)
- moved R7 0.25 mm to (198.0, 91.8)
Connections:
- J13 pad 1: Net-(U1-M1A) -> Net-(U1-M1B)
- J13 pad 2: Net-(U1-M2A) -> Net-(U1-M1A)
- J13 pad 3: Net-(U1-M1B) -> Net-(U1-M2A)
- J14 pad 1: Net-(U2-M1A) -> Net-(U2-M1B)
- J14 pad 2: Net-(U2-M2A) -> Net-(U2-M1A)
- J14 pad 3: Net-(U2-M1B) -> Net-(U2-M2A)
Routing:
- net /LimitSense: track 0.00 -> 145.5 mm, vias 0 -> 2
- net Net-(J9-Pad2): track 0.00 -> 14.2 mm
- net /RADIO CLK: track 68.6 -> 56.1 mm, vias 2 -> 1
- net GND: track 0.00 -> 5.94 mm, vias 5 -> 7
- net Net-(J12-Pad2): track 0.00 -> 5.83 mm
- net Net-(J11-Pad2): track 0.00 -> 5.41 mm
- net Net-(U1-M1B): track 10.1 -> 8.24 mm
- net Net-(U2-M1A): track 18.1 -> 19.3 mm, vias 0 -> 1
- net Net-(U1-M2A): track 9.31 -> 8.27 mm
- net Net-(U1-M1A): track 9.29 -> 8.25 mm
- net +3.3V: track 254.0 -> 254.9 mm
- net Net-(U2-M2B): track 15.6 -> 16.3 mm
Other:
- board text added: "I2C #1"
- board text added: "I2C #2"
- board text added: "Rocket Spatial Position & Orientation Tracker"
