File: Boards/GSat/GSat board/GSat board.kicad_sch (KiCad schematic)
At the start: 60 parts, among them IC1 LTC4418IUF#PBF, IC2 MCP23017-E_SP, J1 B3B-XH-A_LF__SN_, J10 Conn_01x05_Pin, J11 Conn_01x06_Pin, J12 XT30UPB-F, J13 B4B-XH-A_LF__SN_, J14 B4B-XH-A_LF__SN_, J15 B4B-XH-A_LF__SN_, J16 B4B-XH-A_LF__SN_, J2 XT30UPB-F, J3 B3B-XH-A_LF__SN_, J4 B3B-XH-A_LF__SN_, J9 Conn_01x02_Pin, Q1 PMOS, Q2 PMOS, Q3 PMOS, Q4 PMOS, U1 TMC2209_SILENTSTEPSTICK, U10 ST1L05APU33R, U2 TMC2209_SILENTSTEPSTICK, U3 E28-2G4M27SX, U4 E28-2G4M27SX, U5 MAX485_MODULE_5V_LOGIC_TLL_TO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

Commit message: Revert "GSPOT"
This reverts commit 8c379314ca4fbea904d10af8cef34905ce442d4e.
Parts:
- removed J1, J3, J4: B3B-XH-A_LF__SN_, B3BXHALFSN, symbol B3B-XH-A_LF__SN_:B3B-XH-A_LF__SN_
- added J6, J7, J8: Conn_01x03_Pin, symbol Connector:Conn_01x03_Pin
- added TP5: TestPoint, TestPoint:TestPoint_Pad_2.0x2.0mm, symbol Connector:TestPoint
Connections:
- net +3.3V IC is gone; now on net +3.3V: C39.2, TP2.1, U1.16 (~{EN}), U1.2 (VIO), U10.2 (V0), U2.16 (~{EN}), U2.2 (VIO)
- net +24V: now also TP5.1
- net +3.3V: now also J6.3 (Pin_3), J7.3 (Pin_3), J8.3 (Pin_3)
- net GND: now also J6.1 (Pin_1), J7.1 (Pin_1), J8.1 (Pin_1); no longer A1.33 (AGND)
- net LimitSwitch1: now also J6.2 (Pin_2)
- net LimitSwitch2: now also J7.2 (Pin_2)
- net LimitSwitch3: now also J8.2 (Pin_2)
- no-connect marks 22 -> 17
