File: Boards/GSat/GSat board/GSat board.kicad_sch (KiCad schematic)
At the start: 64 parts, among them IC1 LTC4418IUF#PBF, IC2 MCP23017-E_SP, IC3 SP3485CN-L_TR, J1 B3B-XH-A_LF__SN_, J10 Conn_01x05_Pin, J11 Conn_01x06_Pin, J12 XT30UPB-F, J13 B4B-XH-A_LF__SN_, J14 B4B-XH-A_LF__SN_, J15 B4B-XH-A_LF__SN_, J16 B4B-XH-A_LF__SN_, J2 XT30UPB-F, J3 B3B-XH-A_LF__SN_, J4 B3B-XH-A_LF__SN_, J9 Conn_01x02_Pin, Q1 PMOS, Q2 PMOS, Q3 PMOS, Q4 PMOS, U1 TMC2209_SILENTSTEPSTICK, U10 ST1L05APU33R, U2 TMC2209_SILENTSTEPSTICK, U3 E28-2G4M27SX, U4 E28-2G4M27SX, U5 MAX485_MODULE_5V_LOGIC_TLL_TO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

Commit message: GSAT REORGANIZED AND TRACED (mostly)
insert here the entire shrek script
Parts:
- removed C37, C39: 4.7uF, Capacitor-0402:Capacitor_0402, symbol Device:C
- removed C40: 1uF, Capacitor-0402:Capacitor_0402, symbol Device:C
- removed C41: 1nF, Capacitor-0402:Capacitor_0402, symbol Device:C
- removed C42, C43, C44, C45, C46: 100nF, Capacitor-0402:Capacitor_0402, symbol Device:C
- removed C47: 220uF, Capacitor-0402:Capacitor_0402, symbol Device:C
- removed D1, D2: SMBJ24CA, SMBJ24CA:DIOM5436X244N, symbol SMBJ24CA:SMBJ24CA
- removed F1, F2: 0ABB-6000-TM, 0ABB-6000-TM:0ABB6000TM, symbol 0ABB-6000-TM:0ABB-6000-TM
- removed IC1: LTC4418IUF#PBF, LTC4418:QFN50P400X400X80-21N-D, symbol LTC4418IUF#PBF:LTC4418IUF#PBF
- removed J12, J2: XT30UPB-F, XT30UPB-F:XT30UPBF, symbol XT30UPB-F:XT30UPB-F
- removed J9: Conn_01x02_Pin, symbol Connector:Conn_01x02_Pin
- removed Q1, Q2, Q3, Q4: PMOS, Package_TO_SOT_SMD:TO-252-3_TabPin2, symbol Simulation_SPICE:PMOS
- removed R1: 1K, Resistor_SMD:R_0603_1608Metric_Pad0.98x0.95mm_HandSolder, symbol Device:R
- removed R10, R5: 9.31K, Resistor_SMD:R_0603_1608Metric_Pad0.98x0.95mm_HandSolder, symbol Device:R
- removed R15, R7: 39.6K, Resistor_SMD:R_0603_1608Metric_Pad0.98x0.95mm_HandSolder, symbol Device:R
- removed R3: 10K, Resistor_SMD:R_0603_1608Metric_Pad0.98x0.95mm_HandSolder, symbol Device:R
- removed R4, R9: 1M, Resistor_SMD:R_0603_1608Metric_Pad0.98x0.95mm_HandSolder, symbol Device:R
- removed TP2, TP3, TP4: TestPoint, TestPoint:TestPoint_Pad_2.0x2.0mm, symbol Connector:TestPoint
- removed U10: ST1L05APU33R, LDO ST1L05A:DFN_5APU33R_STM, symbol LDO_ST1L05A:ST1L05APU33R
- removed U4: E28-2G4M27SX, Radio_Module_PST:Radio_Module_PST, symbol E28-2G4M27S:E28-2G4M27SX
- removed U5: MAX485_MODULE_5V_LOGIC_TLL_TO_RS-485_CONVERTER, MAX485Module:MODULE_MAX485_MODULE_5V_LOGIC_TLL_TO_RS-485_CONVERTER, symbol MAX485_MODULE_5V_LOGIC_TLL_TO_RS-485_CONVERTER:MAX485_MODULE_5V_LOGIC_TLL_TO_RS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
- added J5: 1723163304, 1723163304:MOLEX_1723163304, symbol 1723163304:1723163304
- added U4: LD1117S33TR_SOT223, Package_TO_SOT_SMD:SOT-223-3_TabPin2, symbol Regulator_Linear:LD1117S33TR_SOT223
- C4, C5: footprint Capacitor-0402:Capacitor_0402 -> Capacitor_SMD:C_0603_1608Metric_Pad1.08x0.95mm_HandSolder
- IC3: footprint SOIC127P600X175-8N -> SP3485CN-L_TR:SOIC127P600X175-8N
- J1, J3, J4: footprint B3BXHALFSN -> B3B-XH-A_LF__SN:B3BXHALFSN
- J13, J14, J15, J16: footprint B4BXHALFSN -> B4B-XH-A_LF__SN_:B4BXHALFSN
- R11, R12, R13, R14, R6, R8: footprint Resistor-0402:RES_0402 -> Resistor_SMD:R_0603_1608Metric_Pad0.98x0.95mm_HandSolder
Connections:
- net +3.3V IC is gone; now on net +3.3V: U1.16 (~{EN}), U1.2 (VIO), U2.16 (~{EN}), U2.2 (VIO)
- net CS_OMNI is gone; now on net EXP INTERRUPT: A1.22 (GPIO17)
- net +24V: now also J5.1
- net +3.3V: now also U4.2 (VO); no longer A1.36 (3V3)
- net +5V: now also U4.3 (VI)
- net GND: now also J5.2, U4.1 (GND)
- net RS_A: now also J5.4
- net RS_B: now also J5.3
- net OMNI_BUSY: no longer names the net of A1.27 (GPIO21)
- net OMNI_DIO1: no longer names the net of A1.29 (GPIO22)
- net OMNI_NRESET: no longer names the net of IC2.26 (GPA5)
- net OMNI_RX_EN: no longer names the net of IC2.27 (GPA6)
- net OMNI_TX_EN: no longer names the net of IC2.28 (GPA7)
- no-connect marks 22 -> 18
Other:
- note added: "Lista de melhoramentos: -mudar ldo para o https://mauser.pt/001-9136/regulador-de-tensao-ld1117v33-3-3v-0-8a"
- note removed: "Conectores TODOS"
- note removed: "Lista de melhoramentos: -retirar o conectores todos -trocar footprints 0402 e 0603 para algo maior -separar o radio em dois canais de spi -mudar do max485 para o sp3485 -mudar ldo para o https://mauser.pt/001-9136/regulador-de-tensao-ld1117v33-3-3v-0-8a"
- moved on the sheet: R2, U3

Commit message: GSPOT update
Parts:
- removed C4, C5: 100n, Capacitor_SMD:C_0603_1608Metric_Pad1.08x0.95mm_HandSolder, symbol Device:C_Small
- removed J11: Conn_01x06_Pin, Connector_PinSocket_2.54mm:PinSocket_1x06_P2.54mm_Vertical, symbol Connector:Conn_01x06_Pin
- removed R6, R8: 1k, Resistor_SMD:R_0603_1608Metric_Pad0.98x0.95mm_HandSolder, symbol Device:R
- added A2: RaspberryPi_Pico, Module:RaspberryPi_Pico_Common_Unspecified, symbol MCU_Module:RaspberryPi_Pico
- added C1, C2, C3: 100n, Capacitor_SMD:C_0603_1608Metric_Pad1.08x0.95mm_HandSolder, symbol Device:C
- added C44: 470u, Capacitor_SMD:CP_Elec_10x10, symbol Device:C
- added C7, C9: 100u, Capacitor_SMD:CP_Elec_6.3x7.7, symbol Device:C_Small
- added D1: D_Zener, Diode_SMD:D_SMB, symbol Device:D_Zener
- added F1: 0ABB-6000-TM, 0ABB-6000-TM:0ABB6000TM, symbol 0ABB-6000-TM:0ABB-6000-TM
- added R7, R9: 10k, Resistor_SMD:R_0603_1608Metric_Pad0.98x0.95mm_HandSolder, symbol Device:R
Connections:
- net +3.3V: now also R7.2, R9.2; no longer U1.16 (~{EN}), U2.16 (~{EN})
- net +5V: now also A2.39 (VSYS)
- net CS_UNI: now also A2.22 (GPIO17)
- net Driver1 Dir: now also A2.27 (GPIO21)
- net Driver1 MS1: now also A2.16 (GPIO12)
- net Driver1 MS2: now also A2.17 (GPIO13)
- net Driver1 Step: now also A2.4 (GPIO2)
- net Driver2 Dir: now also A2.26 (GPIO20)
- net Driver2 MS1: now also A2.19 (GPIO14)
- net Driver2 MS2: now also A2.20 (GPIO15)
- net Driver2 Step: now also A2.5 (GPIO3)
- net GND: now also A2.13 (GND), A2.18 (GND), A2.23 (GND), A2.28 (GND), A2.3 (GND), A2.33 (AGND), A2.38 (GND), A2.8 (GND), C1.2, C2.2, C3.2, C44.2, C7.2, C9.2, D1.2 (A); no longer A1.35 (ADC_VREF)
- net GPS PPS: no longer A1.34 (GPIO28_ADC2)
- net GPS RX UART: now also A2.1 (GPIO0)
- net GPS TX UART: now also A2.2 (GPIO1)
- net I2C#1 SCL: now also A2.7 (GPIO5)
- net I2C#1 SDA: now also A2.6 (GPIO4)
- net LimitSwitch1: now also A2.34 (GPIO28_ADC2)
- net LimitSwitch2: now also A2.32 (GPIO27_ADC1)
- net LimitSwitch3: now also A2.31 (GPIO26_ADC0)
- net RADIO CLK: now also A2.24 (GPIO18)
- net RADIO MISO: now also A2.21 (GPIO16)
- net RADIO MOSI: now also A2.25 (GPIO19)
- net RS_ENABLE: now also A2.29 (GPIO22)
- net RS_RX: now also A2.12 (GPIO9)
- net RS_TX: now also A2.11 (GPIO8)
- net UNI_BUSY: now also A2.14 (GPIO10)
- net UNI_DIO1: now also A2.15 (GPIO11)
- net UNI_RX_EN: now also A2.9 (GPIO6)
- net UNI_TX_EN: now also A2.10 (GPIO7)
- net +24V renamed +12V
- net +12V: now also C1.1, C2.1, C3.1, C44.1, C7.1, C9.1, D1.1 (K), F1.1; no longer J5.1
- net CS_MSD: no longer names the net of A1.17 (GPIO13)
- net Driver1 VREF: no longer names the net of A1.31 (GPIO26_ADC0)
- net Driver2 VREF: no longer names the net of A1.32 (GPIO27_ADC1)
- net MSD CLK: no longer names the net of A1.19 (GPIO14)
- net MSD MISO renamed TMC EN
- net TMC EN: now also U1.16 (~{EN}), U2.16 (~{EN}), R7.1, R9.1
- net MSD MOSI: no longer names the net of A1.20 (GPIO15)
- new net: F1.2, J5.1
- no-connect marks 18 -> 27
Other:
- note removed: "Lista de melhoramentos: -mudar ldo para o https://mauser.pt/001-9136/regulador-de-tensao-ld1117v33-3-3v-0-8a"

Commit message: GSPOT PCB (almost final)
apenas finalizar uma feature e detalhes
Parts:
- removed A2: RaspberryPi_Pico, Module:RaspberryPi_Pico_Common_Unspecified, symbol MCU_Module:RaspberryPi_Pico
- removed IC2: MCP23017-E_SP, MCP23017:DIP794W56P254L3486H508Q28N, symbol MCP23017-E_SP:MCP23017-E_SP
- removed J5: 1723163304, 1723163304:MOLEX_1723163304, symbol 1723163304:1723163304
- removed R14: 10k, Resistor_SMD:R_0603_1608Metric_Pad0.98x0.95mm_HandSolder, symbol Device:R
- added C5: 100n, Capacitor_SMD:C_0603_1608Metric_Pad1.08x0.95mm_HandSolder, symbol Device:C
- added J17: B4B-XH-A_LF__SN_, B4B-XH-A_LF__SN_:B4BXHALFSN, symbol B4B-XH-A_LF__SN_:B4B-XH-A_LF__SN_
- added J2: 172298-1104, 1723163304:172298-YY04, symbol 172298-1104:172298-1104
- added J5, J6, J7, J8: B2B-XH-A-M_LF__SN_, B2BXHAMLFSN, symbol B2B-XH-A-M_LF__SN_:B2B-XH-A-M_LF__SN_
- added R20: 1k, Resistor_SMD:R_0603_1608Metric_Pad0.98x0.95mm_HandSolder, symbol Device:R
- added R21: 10k, Resistor_SMD:R_0603_1608Metric_Pad0.98x0.95mm_HandSolder, symbol Device:R
- D1: value D_Zener -> SMAJ14A
- F1: value 0ABB-6000-TM -> 0680L4000-05; footprint 0ABB-6000-TM:0ABB6000TM -> Fuse:Fuse_2512_6332Metric
- R11: value 10k -> 6.8k
- R12: value 10k -> 1k
- R13: value 10k -> 22k
Connections:
- net Driver1 MS1 is gone; now on net GND: U1.15 (MS1)
- net Driver1 MS2 is gone; now on net GND: U1.14 (MS2)
- net Driver2 MS1 is gone; now on net +3.3V: U2.15 (MS1)
- net Driver2 MS2 is gone; now on net GND: U2.14 (MS2)
- net EXP INTERRUPT is gone; now on net I2C#1 SCL: A1.22 (GPIO17)
- net +3.3V: now also J17.1, R21.2; no longer J1.1, J3.1, J4.1, R11.2, R12.2, R13.2
- net +5V: now also J5.1, J7.1
- net CS_UNI: now also A1.7 (GPIO5); no longer A1.26 (GPIO20)
- net Driver1 Dir: now also A1.25 (GPIO19)
- net Driver1 Step: now also A1.20 (GPIO15); no longer A1.4 (GPIO2)
- net Driver2 Dir: now also A1.24 (GPIO18)
- net Driver2 Step: now also A1.15 (GPIO11); no longer A1.5 (GPIO3)
- net GND: now also R11.1, R12.1, R13.1, C5.2, J17.4, J2.2, J6.2, J8.2; no longer J1.3, J3.3, J4.3
- net I2C#1 SCL: now also J17.3; no longer A1.7 (GPIO5), J15.3
- net I2C#1 SDA: now also A1.21 (GPIO16), J17.2; no longer A1.6 (GPIO4), J15.2
- net I2C#2 SCL: now also A1.32 (GPIO27_ADC1), J15.3; no longer A1.10 (GPIO7)
- net I2C#2 SDA: now also A1.31 (GPIO26_ADC0), J15.2; no longer A1.9 (GPIO6)
- net RADIO CLK: now also A1.4 (GPIO2); no longer A1.24 (GPIO18)
- net RADIO MISO: now also A1.6 (GPIO4); no longer A1.21 (GPIO16)
- net RADIO MOSI: now also A1.5 (GPIO3); no longer A1.25 (GPIO19)
- net RS_A: now also J2.4
- net RS_B: now also J2.3
- net RS_ENABLE: now also A1.14 (GPIO10)
- net TMC EN: now also A1.19 (GPIO14); no longer A1.16 (GPIO12)
- net UNI_BUSY: now also A1.29 (GPIO22); no longer A1.14 (GPIO10)
- net UNI_DIO1: now also A1.26 (GPIO20); no longer A1.15 (GPIO11)
- net UNI_NRESET: now also A1.27 (GPIO21)
- net UNI_RX_EN: now also A1.9 (GPIO6)
- net UNI_TX_EN: now also A1.10 (GPIO7)
- net TMC RX UART: now reaches A1.17 (GPIO13)
- net TMC RX UART: now also U1.12 (UART), U2.12 (UART), R20.1
- net LimitSense: now reaches A1.34 (GPIO28_ADC2)
- net LimitSense: now also J1.1, J3.1, J4.1, C5.1, R21.1
- net at F1.2: now also J2.1
- net LimitSwitch1: no longer names the net of J1.2
- net LimitSwitch1: no longer R11.1
- net LimitSwitch2: no longer names the net of J3.2
- net LimitSwitch2: no longer R12.1
- net LimitSwitch3: no longer names the net of J4.2
- net LimitSwitch3: no longer R13.1
- new net: J7.2, J8.1
- new net: J4.3, R13.2
- new net: J3.3, R11.2
- new net: J5.2, J6.1
- new net: J1.3, R12.2
- new net TMC TX UART: A1.16 (GPIO12), R20.2
- no-connect marks 27 -> 19
Other:
- note added: "Magnetometer"
- note removed: "Qual o power dos switches"
- note removed: "Reorientar os pins para ser mais conveniente se for preciso"
- moved on the sheet: C1, C44, D1, F1

Commit message: RSPOT board (FINAL) (?)
Parts:
- removed J1, J3, J4: B3B-XH-A_LF__SN_, B3B-XH-A_LF__SN:B3BXHALFSN, symbol B3B-XH-A_LF__SN_:B3B-XH-A_LF__SN_
- added J11, J12, J9: B2B-XH-A-M_LF__SN_, B2B-XH-A-M_LF__SN_:B2BXHAMLFSN, symbol B2B-XH-A-M_LF__SN_:B2B-XH-A-M_LF__SN_
- C1, C2, C3, C5: footprint Capacitor_SMD:C_0603_1608Metric_Pad1.08x0.95mm_HandSolder -> Capacitor_SMD:C_0805_2012Metric_Pad1.18x1.45mm_HandSolder
- J5, J6, J7, J8: footprint B2BXHAMLFSN -> B2B-XH-A-M_LF__SN_:B2BXHAMLFSN
- R11, R12, R13, R18, R2, R20, R21, R7, R9: footprint Resistor_SMD:R_0603_1608Metric_Pad0.98x0.95mm_HandSolder -> Resistor_SMD:R_0805_2012Metric_Pad1.20x1.40mm_HandSolder
Connections:
- net LimitSense: now also J11.1, J12.1, J9.1
- net at R13.2: now also J12.2
- net at J14.1: now also U2.3 (M1B); no longer U2.4 (M1A)
- net at J14.2: now also U2.4 (M1A); no longer U2.5 (M2A)
- net at J14.3: now also U2.5 (M2A); no longer U2.3 (M1B)
- net at R11.2: now also J11.2
- net at J13.1: now also U1.3 (M1B); no longer U1.4 (M1A)
- net at J13.2: now also U1.4 (M1A); no longer U1.5 (M2A)
- net at J13.3: now also U1.5 (M2A); no longer U1.3 (M1B)
- net at R12.2: now also J9.2
- no-connect marks 19 -> 16
Other:
- moved on the sheet: J14
